File: EDA/TrailCurrentHeadwatersCM5Carrier/TrailCurrentHeadwatersCM5Carrier.kicad_sch (KiCad schematic)
At the start: 12 parts, among them J11 USB_C_Receptacle_USB2.0

Commit message: Carrier board updated to point to items brought into our own libraries
Parts:
- H1, H2, H3, H4, H5, H6, H7, H8: footprint TrailCurrentHeadwatersCM5Carrier:MountingHole_2.7mm_M2.5_DIN965 -> TrailCurrentFootprints:MountingHole_2.7mm_M2.5_DIN965
Changed lines of the file:
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@@
 			)
 		)
-		(property "Footprint" "TrailCurrentHeadwatersCM5Carrier:MountingHole_2.7mm_M2.5_DIN965"
+		(property "Footprint" "TrailCurrentFootprints:MountingHole_2.7mm_M2.5_DIN965"
 			(at 22.86 180.975 0)
 			(effects
@@
 		)
 		(instances
-			(project "TrailCurrentHeadwatersCM5Carrier"
+			(project "TrailCurrentSymbolLibrary"
 				(path "/e63e39d7-6ac0-4ffd-8aa3-1841a4541b55"
 					(reference "H4")
@@
 			)
 		)
-		(property "Footprint" "TrailCurrentHeadwatersCM5Carrier:MountingHole_2.7mm_M2.5_DIN965"
+		(property "Footprint" "TrailCurrentFootprints:MountingHole_2.7mm_M2.5_DIN965"
 			(at 22.86 175.895 0)
 			(effects
@@
 		)
 		(instances
-			(project "TrailCurrentHeadwatersCM5Carrier"
+			(project "TrailCurrentSymbolLibrary"
 				(path "/e63e39d7-6ac0-4ffd-8aa3-1841a4541b55"
 					(reference "H3")
@@
 			)
 		)
-		(property "Footprint" "TrailCurrentHeadwatersCM5Carrier:MountingHole_2.7mm_M2.5_DIN965"
+		(property "Footprint" "TrailCurrentFootprints:MountingHole_2.7mm_M2.5_DIN965"
 			(at 22.86 170.815 0)
 			(effects
@@
 		)
 		(instances
-			(project "TrailCurrentHeadwatersCM5Carrier"
+			(project "TrailCurrentSymbolLibrary"
 				(path "/e63e39d7-6ac0-4ffd-8aa3-1841a4541b55"
 					(reference "H2")
@@
 			)
 		)
-		(property "Footprint" "TrailCurrentHeadwatersCM5Carrier:MountingHole_2.7mm_M2.5_DIN965"
+		(property "Footprint" "TrailCurrentFootprints:MountingHole_2.7mm_M2.5_DIN965"
 			(at 22.86 165.735 0)
 			(effects
@@
 		)
 		(instances
-			(project "TrailCurrentHeadwatersCM5Carrier"
+			(project "TrailCurrentSymbolLibrary"
 				(path "/e63e39d7-6ac0-4ffd-8aa3-1841a4541b55"
 					(reference "H1")
@@
 			)
 		)
-		(property "Footprint" "TrailCurrentHeadwatersCM5Carrier:MountingHole_2.7mm_M2.5_DIN965"
+		(property "Footprint" "TrailCurrentFootprints:MountingHole_2.7mm_M2.5_DIN965"
 			(at 43.815 165.735 0)
 			(effects
@@
 		)
 		(instances
-			(project "TrailCurrentHeadwatersCM5Carrier"
+			(project "TrailCurrentSymbolLibrary"
 				(path "/e63e39d7-6ac0-4ffd-8aa3-1841a4541b55"
 					(reference "H5")
@@
 			)
 		)
-		(property "Footprint" "TrailCurrentHeadwatersCM5Carrier:MountingHole_2.7mm_M2.5_DIN965"
+		(property "Footprint" "TrailCurrentFootprints:MountingHole_2.7mm_M2.5_DIN965"
 			(at 43.815 180.975 0)
 			(effects
@@
 		)
 		(instances
-			(project "TrailCurrentHeadwatersCM5Carrier"
+			(project "TrailCurrentSymbolLibrary"
 				(path "/e63e39d7-6ac0-4ffd-8aa3-1841a4541b55"
 					(reference "H8")
@@
 			)
 		)
-		(property "Footprint" "TrailCurrentHeadwatersCM5Carrier:MountingHole_2.7mm_M2.5_DIN965"
+		(property "Footprint" "TrailCurrentFootprints:MountingHole_2.7mm_M2.5_DIN965"
 			(at 43.815 175.895 0)
 			(effects
@@
 		)
 		(instances
-			(project "TrailCurrentHeadwatersCM5Carrier"
+			(project "TrailCurrentSymbolLibrary"
 				(path "/e63e39d7-6ac0-4ffd-8aa3-1841a4541b55"
 					(reference "H7")
@@
 			)
 		)
-		(property "Footprint" "TrailCurrentHeadwatersCM5Carrier:MountingHole_2.7mm_M2.5_DIN965"
+		(property "Footprint" "TrailCurrentFootprints:MountingHole_2.7mm_M2.5_DIN965"
 			(at 43.815 170.815 0)
 			(effects
@@
 		)
 		(instances
-			(project "TrailCurrentHeadwatersCM5Carrier"
+			(project "TrailCurrentSymbolLibrary"
 				(path "/e63e39d7-6ac0-4ffd-8aa3-1841a4541b55"
 					(reference "H6")
@@
 		)
 		(instances
-			(project "TrailCurrentHeadwatersCM5Carrier"
+			(project "TrailCurrentSymbolLibrary"
 				(path "/e63e39d7-6ac0-4ffd-8aa3-1841a4541b55"
 					(reference "#PWR031")
@@
 		)
 		(instances
-			(project "TrailCurrentHeadwatersCM5Carrier"
+			(project "TrailCurrentSymbolLibrary"
 				(path "/e63e39d7-6ac0-4ffd-8aa3-1841a4541b55"
 					(reference "C18")
@@
 		)
 		(instances
-			(project "TrailCurrentHeadwatersCM5Carrier"
+			(project "TrailCurrentSymbolLibrary"
 				(path "/e63e39d7-6ac0-4ffd-8aa3-1841a4541b55"
 					(reference "J11")
@@
 		)
 		(instances
-			(project "TrailCurrentHeadwatersCM5Carrier"
+			(project "TrailCurrentSymbolLibrary"
 				(path "/e63e39d7-6ac0-4ffd-8aa3-1841a4541b55"
 					(reference "R9")
@@
 		)
 		(instances
-			(project "TrailCurrentHeadwatersCM5Carrier"
+			(project "TrailCurrentSymbolLibrary"
 				(path "/e63e39d7-6ac0-4ffd-8aa3-1841a4541b55"
 					(reference "C9")
@@
 		)
 		(instances
-			(project "TrailCurrentHeadwatersCM5Carrier"
+			(project "TrailCurrentSymbolLibrary"
 				(path "/e63e39d7-6ac0-4ffd-8aa3-1841a4541b55"
 					(reference "#PWR02")
@@
 		)
 		(instances
-			(project "TrailCurrentHeadwatersCM5Carrier"
+			(project "TrailCurrentSymbolLibrary"
 				(path "/e63e39d7-6ac0-4ffd-8aa3-1841a4541b55"
 					(reference "#PWR013")
@@
 		)
 		(instances
-			(project "TrailCurrentHeadwatersCM5Carrier"
+			(project "TrailCurrentSymbolLibrary"
 				(path "/e63e39d7-6ac0-4ffd-8aa3-1841a4541b55"
 					(page "3")
@@
 		)
 		(instances
-			(project "TrailCurrentHeadwatersCM5Carrier"
+			(project "TrailCurrentSymbolLibrary"
 				(path "/e63e39d7-6ac0-4ffd-8aa3-1841a4541b55"
 					(page "2")
@@
 		)
 		(instances
-			(project "TrailCurrentHeadwatersCM5Carrier"
+			(project "TrailCurrentSymbolLibrary"
 				(path "/e63e39d7-6ac0-4ffd-8aa3-1841a4541b55"
 					(page "4")
