File: EDA/TrailCurrentHeadwatersCM5Carrier/TrailCurrentHeadwatersCM5Carrier_HighSpeed.kicad_sch (KiCad schematic)
At the start: 19 parts, among them J10 690-019-298-412, J12 USB3_A, J16 Conn_01x22_Female, J22 690-019-298-412, J5 Conn_01x22_Female, J6 THD-02-R, U12 RT9742SNGV, U6 AP22653W6

Commit message: Carrier board updated to point to items brought into our own libraries
Parts:
- J10, J22: footprint TrailCurrentHeadwatersCM5Carrier:EDAC 690-019-298-412 -> TrailCurrentFootprints:EDAC 690-019-298-412; symbol TrailCurrentHeadwatersCM5Carrier:HDMI_A_1.4 -> TrailCurrentSymbolLibrary:HDMI_A_1.4
- J12: footprint TrailCurrentHeadwatersCM5Carrier:MTCONN_UBAF30-D2011 -> TrailCurrentFootprints:MTCONN_UBAF30-D2011; symbol TrailCurrentHeadwatersCM5Carrier:USB3_A -> TrailCurrentSymbolLibrary:USB3_A
- J16, J5: footprint TrailCurrentHeadwatersCM5Carrier:Hirose_FH12-22S-0.5SH_1x22-1MP_P0.50mm_Horizontal -> TrailCurrentFootprints:Hirose_FH12-22S-0.5SH_1x22-1MP_P0.50mm_Horizontal
- Module1: footprint TrailCurrentHeadwatersCM5Carrier:Raspberry-Pi-5-Compute-Module -> TrailCurrentFootprints:Raspberry-Pi-5-Compute-Module; symbol TrailCurrentHeadwatersCM5Carrier:ComputeModule5-CM5 -> TrailCurrentSymbolLibrary:ComputeModule5-CM5
- U12: symbol TrailCurrentHeadwatersCM5Carrier:RT9742SNGV -> TrailCurrentSymbolLibrary:RT9742SNGV
- U6: symbol TrailCurrentHeadwatersCM5Carrier:AP2553W6 -> TrailCurrentSymbolLibrary:AP2553W6
