File: EDA/TrailCurrentHeadwatersCM5Carrier/TrailCurrentHeadwatersCM5Carrier_PCIeM2.kicad_sch (KiCad schematic)
At the start: 24 parts, among them J4 Bus_M.2_Socket_M, M1 M.2 Screw, M2 M.2 Solder Nut, M3 M.2 Solder Nut, M4 M.2 Solder Nut, M5 M.2 Solder Nut, U7 ASEK-32.768KHZ-L-R-T, U8 AP3441SHE-7B

Commit message: Carrier board updated to point to items brought into our own libraries
Parts:
- J4: footprint TrailCurrentHeadwatersCM5Carrier:M.2 M Key socket -> TrailCurrentFootprints:M.2 M Key socket; symbol TrailCurrentHeadwatersCM5Carrier:Bus_M.2_Socket_M -> TrailCurrentSymbolLibrary:Bus_M.2_Socket_M
- L1: footprint TrailCurrentHeadwatersCM5Carrier:L_Bourns_SRP5030CC -> TrailCurrentFootprints:L_Bourns_SRP5030CC
- M1: symbol TrailCurrentHeadwatersCM5Carrier:M.2_Screw -> TrailCurrentSymbolLibrary:M.2_Screw
- M2, M3, M4, M5: symbol TrailCurrentHeadwatersCM5Carrier:SolderNut -> TrailCurrentSymbolLibrary:SolderNut
- U7: symbol TrailCurrentHeadwatersCM5Carrier:ASEK-32.768KHZ-L-R-T -> TrailCurrentSymbolLibrary:ASEK-32.768KHZ-L-R-T
- U8: symbol TrailCurrentHeadwatersCM5Carrier:AP3441SHE-7B -> TrailCurrentSymbolLibrary:AP3441SHE-7B
